File: HarwinHVv2board.sch (KiCad schematic (older format))
At the start: 7 parts, among them J1 HV2, J2 GND2, J3 HarwinHV1, J4 HarwinHV2, J5 HarwinGND, J6 HV1, J7 GND1

Commit message: Changed Harwin connector pads to 1.3mm drill hole on a 5.75 x 2 mm rectangular pad with rounded corners.
Parts:
- J3, J4, J5: footprint Connector_Wire:SolderWire-0.75sqmm_1x01_D1.25mm_OD2.3mm -> HarwinHVv2board:Pin_D1.3mm_L5.75mmW2.0mm
Changed lines of the file:
@@
 F 0 "J3" V 6038 2162 50  0000 R CNN
 F 1 "HarwinHV1" V 5947 2162 50  0000 R CNN
-F 2 "Connector_Wire:SolderWire-0.75sqmm_1x01_D1.25mm_OD2.3mm" H 6100 2250 50  0001 C CNN
+F 2 "HarwinHVv2board:Pin_D1.3mm_L5.75mmW2.0mm" H 6100 2250 50  0001 C CNN
 F 3 "~" H 6100 2250 50  0001 C CNN
 	1    6100 2250
@@
 F 0 "J4" V 6038 2562 50  0000 R CNN
 F 1 "HarwinHV2" V 6150 2950 50  0000 R CNN
-F 2 "Connector_Wire:SolderWire-0.75sqmm_1x01_D1.25mm_OD2.3mm" H 6100 2650 50  0001 C CNN
+F 2 "HarwinHVv2board:Pin_D1.3mm_L5.75mmW2.0mm" H 6100 2650 50  0001 C CNN
 F 3 "~" H 6100 2650 50  0001 C CNN
 	1    6100 2650
@@
 F 0 "J5" V 6038 3012 50  0000 R CNN
 F 1 "HarwinGND" V 6150 3400 50  0000 R CNN
-F 2 "Connector_Wire:SolderWire-0.75sqmm_1x01_D1.25mm_OD2.3mm" H 6100 3100 50  0001 C CNN
+F 2 "HarwinHVv2board:Pin_D1.3mm_L5.75mmW2.0mm" H 6100 3100 50  0001 C CNN
 F 3 "~" H 6100 3100 50  0001 C CNN
 	1    6100 3100
